File: Manufacuring_drawings/PCB111000_1_V2_CC.brd (EAGLE design)
At the start: 69.9 x 39.9 mm, 37 parts, among them IC1 ATTINY1606, IC2 MEGA8-P, Q1 BSS138, SW1 NO_SW, SW3 NO_PB_1, SW4 NO_PB_1, SW5 NO_PB_1

Commit message: Update PCB111000_1_V2_CC.brd
Parts:
- moved R24 6.10 mm to (16.5, 73.4)
- moved R1 0.90 mm to (25.9, 68.3)
Routing:
- net 0V: track 200.2 -> 181.5 mm, vias 2 -> 7
- net N$14: track 31.3 -> 48.1 mm
- net SEVEN_SEG0: track 54.6 -> 63.2 mm
- net DISPLAY_DRIVER0: track 31.0 -> 36.9 mm
- net DIGIT2: track 21.7 -> 25.1 mm
- net DIGIT7: track 34.5 -> 37.3 mm
- net SEVEN_SEG5: track 61.3 -> 64.1 mm
- net SEVEN_SEG1: track 66.0 -> 68.4 mm
- net N$40: track 43.2 -> 45.3 mm
- net N$8: track 5.07 -> 7.25 mm
- net DISPLAY_DRIVER3: track 32.9 -> 34.8 mm
- net DIGIT0: track 62.7 -> 64.5 mm
- net N$3: track 10.8 -> 12.5 mm
- net SEVEN_SEG6: track 57.8 -> 59.4 mm
- net N$10: track 22.6 -> 24.2 mm
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
Commit message: Update PCB111000_1_V2_CC.brd
Parts:
- moved U$1 12.5 mm to (65.3, 56.4)
Routing:
- net N$17: track 2.44 -> 15.9 mm
- net N$12: track 2.44 -> 11.0 mm
- net DIGIT5: track 31.5 -> 34.6 mm
- net DISPLAY_DRIVER5: track 23.0 -> 26.1 mm
- net N$6: track 33.0 -> 34.4 mm
- net N$10: track 24.2 -> 25.5 mm
- net DISPLAY_DRIVER6: track 27.6 -> 28.3 mm

Commit message: Update PCB111000_1_V2_CC.brd
Parts:
- moved U$1 2.18 mm to (63.5, 57.7), turned to 0 degrees
Routing:
- net N$17: track 15.9 -> 20.5 mm
- net N$10: track 25.5 -> 28.5 mm
- net 0V: track 181.7 -> 183.1 mm
- net SEVEN_SEG6: track 59.4 -> 58.9 mm
Changed lines of the file:
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@@
 <attribute name="VALUE" x="20.854" y="41.985" size="1.27" layer="28" rot="MR90"/>
 </element>
-<element name="U$1" library="mo" package="XTAL" value="XTAL" x="65.278" y="56.388" smashed="yes" rot="R270"/>
+<element name="U$1" library="mo" package="XTAL" value="XTAL" x="63.5" y="57.658" smashed="yes"/>
 </elements>
 <signals>
@@
 <wire x1="55.582" y1="57.277" x2="55.582" y2="59.226" width="0.6096" layer="1"/>
 <wire x1="55.582" y1="59.226" x2="55.372" y2="59.436" width="0.6096" layer="1"/>
-<wire x1="59.055" y1="59.563" x2="59.69" y2="59.563" width="0.6096" layer="1"/>
-<wire x1="77.3938" y1="58.801" x2="79.5528" y2="56.642" width="0.6096" layer="1"/>
-<wire x1="59.69" y1="59.563" x2="60.452" y2="58.801" width="0.6096" layer="1"/>
-<wire x1="60.452" y1="58.801" x2="77.3938" y2="58.801" width="0.6096" layer="1"/>
+<wire x1="76.6318" y1="59.563" x2="79.5528" y2="56.642" width="0.6096" layer="1"/>
 <wire x1="60.85" y1="49.767" x2="60.85" y2="46.167" width="0.6096" layer="1"/>
 <wire x1="58.31" y1="52.307" x2="60.706" y2="49.911" width="0.6096" layer="1"/>
@@
 <wire x1="58.293" y1="56.134" x2="57.15" y2="57.277" width="0.6096" layer="1"/>
 <wire x1="57.15" y1="57.277" x2="55.582" y2="57.277" width="0.6096" layer="1"/>
+<wire x1="59.055" y1="59.563" x2="61.468" y2="59.563" width="0.6096" layer="1"/>
+<wire x1="61.468" y1="59.563" x2="62.611" y2="60.706" width="0.6096" layer="1"/>
+<wire x1="76.1238" y1="59.055" x2="76.6318" y2="59.563" width="0.6096" layer="1"/>
+<wire x1="62.611" y1="60.706" x2="65.786" y2="60.706" width="0.6096" layer="1"/>
+<wire x1="65.786" y1="60.706" x2="67.437" y2="59.055" width="0.6096" layer="1"/>
+<wire x1="67.437" y1="59.055" x2="76.1238" y2="59.055" width="0.6096" layer="1"/>
 </signal>
 <signal name="+5V">
@@
 <wire x1="30.861" y1="66.5226" x2="30.868" y2="66.852" width="0.381" layer="16"/>
 <wire x1="77.1787" y1="62.8721" x2="77.1787" y2="62.5737" width="0.381" layer="1"/>
-<wire x1="77.1787" y1="62.5737" x2="75.819" y2="61.214" width="0.381" layer="1"/>
-<wire x1="66.04" y1="61.214" x2="75.819" y2="61.214" width="0.381" layer="1"/>
-<wire x1="63.1317" y1="64.1223" x2="66.04" y2="61.214" width="0.381" layer="1"/>
-<wire x1="26.67" y1="64.1223" x2="63.1317" y2="64.1223" width="0.381" layer="1"/>
+<wire x1="77.1787" y1="62.5737" x2="76.073" y2="61.468" width="0.381" layer="1"/>
+<wire x1="68.072" y1="61.468" x2="76.073" y2="61.468" width="0.381" layer="1"/>
+<wire x1="65.4177" y1="64.1223" x2="68.072" y2="61.468" width="0.381" layer="1"/>
+<wire x1="26.67" y1="64.1223" x2="65.4177" y2="64.1223" width="0.381" layer="1"/>
 <wire x1="26.67" y1="64.1223" x2="26.1779" y2="63.6302" width="0.381" layer="1"/>
 <wire x1="26.1779" y1="62.9245" x2="26.1779" y2="63.6302" width="0.381" layer="1"/>
@@
 <contactref element="7_SEG2" pad="P$1"/>
 <contactref element="R21" pad="P$1"/>
-<wire x1="70.9803" y1="64.8081" x2="70.9803" y2="66.5226" width="0.381" layer="16"/>
-<wire x1="69.2658" y1="63.0936" x2="70.9803" y2="64.8081" width="0.381" layer="16"/>
+<wire x1="70.9803" y1="64.4271" x2="70.9803" y2="66.5226" width="0.381" layer="16"/>
+<wire x1="69.482740625" y1="62.929540625" x2="70.9803" y2="64.4271" width="0.381" layer="16"/>
 <wire x1="70.9803" y1="66.5226" x2="71.227" y2="66.791" width="0.381" layer="16"/>
-<wire x1="69.2658" y1="63.0936" x2="69.5587" y2="62.8721" width="0.381" layer="16"/>
+<wire x1="69.482740625" y1="62.929540625" x2="69.5587" y2="62.8721" width="0.381" layer="16"/>
 <wire x1="20.574" y1="60.6552" x2="18.5579" y2="62.6713" width="0.381" layer="1"/>
 <wire x1="18.5579" y1="62.9245" x2="18.5579" y2="62.6713" width="0.381" layer="1"/>
 <wire x1="60.6425" y1="61.0362" x2="60.2615" y2="60.6552" width="0.381" layer="1"/>
 <wire x1="60.2615" y1="60.6552" x2="20.574" y2="60.6552" width="0.381" layer="1"/>
-<wire x1="67.5513" y1="61.0362" x2="60.6425" y2="61.0362" width="0.381" layer="16"/>
-<wire x1="69.2658" y1="62.7507" x2="67.5513" y2="61.0362" width="0.381" layer="16"/>
+<wire x1="68.3133" y1="61.7982" x2="61.4045" y2="61.7982" width="0.381" layer="16"/>
+<wire x1="61.4045" y1="61.7982" x2="60.6425" y2="61.0362" width="0.381" layer="16"/>
+<wire x1="69.2658" y1="62.7507" x2="68.3133" y2="61.7982" width="0.381" layer="16"/>
 <wire x1="69.2658" y1="62.7507" x2="69.5587" y2="62.8721" width="0.381" layer="16"/>
 <via x="60.6425" y="61.0362" extent="1-16" drill="0.6096"/>
@@
 <wire x1="58.8137" y1="61.722" x2="29.2481" y2="61.722" width="0.381" layer="1"/>
 <wire x1="59.5376" y1="62.4459" x2="58.8137" y2="61.722" width="0.381" layer="1"/>
-<wire x1="62.3824" y1="62.4459" x2="59.5376" y2="62.4459" width="0.381" layer="1"/>
-<wire x1="64.9351" y1="59.8932" x2="62.3824" y2="62.4459" width="0.381" layer="1"/>
-<wire x1="76.6953" y1="59.8932" x2="64.9351" y2="59.8932" width="0.381" layer="1"/>
-<wire x1="79.5528" y1="62.7507" x2="76.6953" y2="59.8932" width="0.381" layer="1"/>
+<wire x1="65.5574" y1="62.4459" x2="59.5376" y2="62.4459" width="0.381" layer="1"/>
+<wire x1="67.4751" y1="60.5282" x2="65.5574" y2="62.4459" width="0.381" layer="1"/>
+<wire x1="77.3303" y1="60.5282" x2="67.4751" y2="60.5282" width="0.381" layer="1"/>
+<wire x1="79.5528" y1="62.7507" x2="77.3303" y2="60.5282" width="0.381" layer="1"/>
 <wire x1="79.5528" y1="62.7507" x2="79.7187" y2="62.8721" width="0.381" layer="1"/>
 </signal>
@@
 <contactref element="IC2" pad="18"/>
 <contactref element="IC1" pad="P$18"/>
-<wire x1="68.47" y1="53.787" x2="68.47" y2="57.2854" width="0.381" layer="16"/>
-<wire x1="68.47" y1="57.2854" x2="67.8688" y2="57.8866" width="0.381" layer="16"/>
-<wire x1="58.8264" y1="57.8866" x2="67.8688" y2="57.8866" width="0.381" layer="16"/>
 <wire x1="53.1114" y1="63.8175" x2="53.1114" y2="62.103" width="0.381" layer="16"/>
 <wire x1="53.8861" y1="64.5922" x2="53.1114" y2="63.8175" width="0.381" layer="16"/>
@@
 <wire x1="54.3814" y1="60.833" x2="55.88" y2="60.833" width="0.381" layer="16"/>
 <wire x1="55.88" y1="60.833" x2="58.8264" y2="57.8866" width="0.381" layer="16"/>
+<wire x1="58.8264" y1="57.8866" x2="59.6646" y2="57.8866" width="0.381" layer="16"/>
+<wire x1="62.103" y1="60.325" x2="67.056" y2="60.325" width="0.381" layer="16"/>
+<wire x1="67.056" y1="60.325" x2="68.47" y2="58.911" width="0.381" layer="16"/>
+<wire x1="59.6646" y1="57.8866" x2="62.103" y2="60.325" width="0.381" layer="16"/>
+<wire x1="68.47" y1="58.911" x2="68.47" y2="53.787" width="0.381" layer="16"/>
 </signal>
 <signal name="N$12">
 <contactref element="U$1" pad="P$1"/>
 <contactref element="IC2" pad="9"/>
-<wire x1="64.008" y1="56.388" x2="64.643" y2="55.753" width="0.381" layer="16"/>
-<wire x1="64.643" y1="52.010775" x2="64.2143" y2="51.582075" width="0.381" layer="16"/>
-<wire x1="64.2143" y1="51.582075" x2="64.2143" y2="48.3393" width="0.381" layer="16"/>
+<wire x1="64.2143" y1="48.3393" x2="64.2143" y2="51.582075" width="0.381" layer="16"/>
 <wire x1="63.39" y1="47.515" x2="63.39" y2="46.167" width="0.381" layer="16"/>
-<wire x1="64.643" y1="55.753" x2="64.643" y2="52.010775" width="0.381" layer="16"/>
 <wire x1="64.2143" y1="48.3393" x2="63.39" y2="47.515" width="0.381" layer="16"/>
+<wire x1="64.643" y1="52.010775" x2="64.643" y2="55.626" width="0.381" layer="16"/>
+<wire x1="64.643" y1="55.626" x2="63.881" y2="56.388" width="0.381" layer="16"/>
+<wire x1="63.881" y1="56.388" x2="63.5" y2="56.388" width="0.381" layer="16"/>
+<wire x1="64.2143" y1="51.582075" x2="64.643" y2="52.010775" width="0.381" layer="16"/>
 </signal>
 <signal name="N$17">
@@
 <wire x1="70.104" y1="50.927" x2="69.342" y2="51.689" width="0.381" layer="16"/>
 <wire x1="69.342" y1="51.689" x2="67.183" y2="51.689" width="0.381" layer="16"/>
-<wire x1="67.183" y1="51.689" x2="67.183" y2="55.753" width="0.381" layer="16"/>
-<wire x1="67.183" y1="55.753" x2="66.548" y2="56.388" width="0.381" layer="16"/>
 <wire x1="65.93" y1="46.88" x2="67.437" y2="48.387" width="0.381" layer="16"/>
+<wire x1="67.183" y1="56.642" x2="67.183" y2="51.689" width="0.381" layer="16"/>
+<wire x1="63.5" y1="58.928" x2="64.389" y2="58.928" width="0.381" layer="16"/>
+<wire x1="66.675" y1="56.642" x2="67.183" y2="56.642" width="0.381" layer="16"/>
+<wire x1="64.389" y1="58.928" x2="66.675" y2="56.642" width="0.381" layer="16"/>
 </signal>
 </signals>
