File: Manufacuring_drawings/PCB 111000_CP2102_SM_led/PCB111000_1_V2_CC.sch (EAGLE design)
At the start: 38 parts, among them IC1 ATTINY1606, IC2 MEGA8-P, Q1 BSS138, SW1 NO_SW, SW3 NO_PB_1, SW4 NO_PB_1, SW5 NO_PB_1

Commit message: Update PCB111000_1_V2_CC.sch
Parts:
- added U$3: SM_XTAL, mo:SM_XTAL
Connections:
- net N$12: now also U$3.P$1
- net N$17: now also U$3.P$2
Changed lines of the file:
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@@
 <?xml version="1.0" encoding="utf-8"?>
 <!DOCTYPE eagle SYSTEM "eagle.dtd">
-<eagle version="9.6.2">
+<eagle version="9.5.2">
 <drawing>
 <settings>
@@
 <setting verticaltext="up"/>
 </settings>
-<grid distance="0.05" unitdist="inch" unit="inch" style="lines" multiple="1" display="no" altdistance="0.01" altunitdist="inch" altunit="inch"/>
+<grid distance="0.1" unitdist="inch" unit="inch" style="lines" multiple="1" display="no" altdistance="0.01" altunitdist="inch" altunit="inch"/>
 <layers>
 <layer number="1" name="Top" color="4" fill="1" visible="no" active="no"/>
@@
 <part name="U$1" library="mo" deviceset="XTAL" device=""/>
 <part name="U$2" library="home_library" deviceset="DUAL_SM_LED" device=""/>
+<part name="U$3" library="mo" deviceset="SM_XTAL" device=""/>
 </parts>
 <sheets>
@@
 <instance part="U$1" gate="G$1" x="-63.5" y="43.18" smashed="yes"/>
 <instance part="U$2" gate="G$1" x="78.74" y="55.88" smashed="yes" rot="R180"/>
+<instance part="U$3" gate="G$1" x="-63.5" y="33.02" smashed="yes"/>
 </instances>
 <busses>
@@
 <segment>
 <pinref part="U$1" gate="G$1" pin="P$1"/>
-<wire x1="-50.8" y1="44.45" x2="-35.56" y2="44.45" width="0.1524" layer="91"/>
+<wire x1="-50.8" y1="44.45" x2="-48.26" y2="44.45" width="0.1524" layer="91"/>
+<wire x1="-48.26" y1="44.45" x2="-35.56" y2="44.45" width="0.1524" layer="91"/>
 <wire x1="-35.56" y1="44.45" x2="-35.56" y2="48.26" width="0.1524" layer="91"/>
 <pinref part="IC2" gate="G$1" pin="PB6(XTAL1/TOSC1)"/>
@@
 <wire x1="-30.48" y1="50.8" x2="-30.48" y2="48.26" width="0.1524" layer="91"/>
 <wire x1="-30.48" y1="48.26" x2="-35.56" y2="48.26" width="0.1524" layer="91"/>
+<pinref part="U$3" gate="G$1" pin="P$1"/>
+<wire x1="-50.8" y1="34.29" x2="-48.26" y2="34.29" width="0.1524" layer="91"/>
+<wire x1="-48.26" y1="34.29" x2="-48.26" y2="44.45" width="0.1524" layer="91"/>
+<junction x="-48.26" y="44.45"/>
 </segment>
 </net>
@@
 <pinref part="U$1" gate="G$1" pin="P$2"/>
 <wire x1="-45.72" y1="41.91" x2="-50.8" y2="41.91" width="0.1524" layer="91"/>
-</segment>
-</net>
+<pinref part="U$3" gate="G$1" pin="P$2"/>
+<wire x1="-50.8" y1="31.75" x2="-45.72" y2="31.75" width="0.1524" layer="91"/>
+<wire x1="-45.72" y1="31.75" x2="-45.72" y2="40.64" width="0.1524" layer="91"/>
+<junction x="-45.72" y="40.64"/>
+</segment>
+</net>
