File: Manufacuring_drawings/PCB 111000_CP2102_SM_led/PCB111000_1_V2_CC.brd (EAGLE design)
At the start: 69.9 x 39.9 mm, 38 parts, among them IC1 ATTINY1606, IC2 MEGA8-P, Q1 BSS138, SW1 NO_SW, SW3 NO_PB_1, SW4 NO_PB_1, SW5 NO_PB_1

Commit message: Update PCB111000_1_V2_CC.brd
Parts:
- added U$3: SM_XTAL, mo:SM_XTAL
Connections:
- net N$12: now also U$3.P$1
- net N$17: now also U$3.P$2
Routing:
- net N$12: track 11.4 -> 14.7 mm
- net N$17: track 20.5 -> 23.2 mm
Changed lines of the file:
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@@
 <?xml version="1.0" encoding="utf-8"?>
 <!DOCTYPE eagle SYSTEM "eagle.dtd">
-<eagle version="9.6.2">
+<eagle version="9.5.2">
 <drawing>
 <settings>
@@
 <setting verticaltext="up"/>
 </settings>
-<grid distance="0.005" unitdist="inch" unit="inch" style="lines" multiple="1" display="no" altdistance="0.025" altunitdist="inch" altunit="inch"/>
+<grid distance="0.005" unitdist="inch" unit="mil" style="lines" multiple="1" display="no" altdistance="0.025" altunitdist="inch" altunit="mil"/>
 <layers>
 <layer number="1" name="Top" color="4" fill="1" visible="yes" active="yes"/>
@@
 <param name="mdSmdStop" value="0mil"/>
 <param name="msWidth" value="15mil"/>
-<param name="msDrill" value="22mil"/>
+<param name="msDrill" value="13mil"/>
 <param name="msMicroVia" value="9.99mm"/>
 <param name="msBlindViaRatio" value="0.5"/>
@@
 <element name="U$1" library="mo" package="XTAL" value="XTAL" x="63.5" y="57.658" smashed="yes"/>
 <element name="U$2" library="home_library" package="SM_DUAL_LED" value="DUAL_SM_LED" x="75.692" y="58.801" smashed="yes" rot="R90"/>
+<element name="U$3" library="mo" package="SM_XTAL" value="SM_XTAL" x="61.849" y="43.434" smashed="yes"/>
 </elements>
 <signals>
@@
 <wire x1="60.85" y1="44.392971875" x2="60.85" y2="46.167" width="0.381" layer="16"/>
 <wire x1="60.85" y1="44.392971875" x2="59.6646" y2="42.740825" width="0.381" layer="16"/>
-<wire x1="59.6646" y1="43.348834375" x2="59.6646" y2="41.4909" width="0.381" layer="1"/>
 <wire x1="59.6646" y1="41.4909" x2="59.651" y2="41.453" width="0.381" layer="1"/>
-<wire x1="60.85" y1="45.00098125" x2="59.6646" y2="43.348834375" width="0.381" layer="1"/>
-<wire x1="60.85" y1="45.00098125" x2="60.85" y2="46.167" width="0.381" layer="1"/>
 <wire x1="26.924" y1="57.912" x2="27.051" y2="57.785" width="0.6096" layer="1"/>
 <wire x1="27.051" y1="57.785" x2="27.051" y2="55.626" width="0.6096" layer="1"/>
@@
 <wire x1="61.468" y1="59.563" x2="62.611" y2="60.706" width="0.6096" layer="1"/>
 <wire x1="62.611" y1="60.706" x2="65.786" y2="60.706" width="0.6096" layer="1"/>
-<wire x1="65.786" y1="60.706" x2="66.929" y2="59.563" width="0.6096" layer="1"/>
+<wire x1="65.786" y1="60.706" x2="67.191" y2="59.301" width="0.6096" layer="1"/>
 <wire x1="80.48" y1="57.176" x2="81" y2="57.176" width="0.6096" layer="1"/>
 <wire x1="81" y1="57.176" x2="82.677" y2="55.499" width="0.6096" layer="1"/>
@@
 <contactref element="U$2" pad="P$3"/>
 <contactref element="U$2" pad="P$4"/>
-<wire x1="66.929" y1="59.563" x2="67.191" y2="59.301" width="0.6096" layer="1"/>
 <wire x1="67.191" y1="59.301" x2="73.692" y2="59.301" width="0.6096" layer="1"/>
 <wire x1="73.692" y1="59.301" x2="73.692" y2="57.801" width="0.6096" layer="1"/>
@@
 <wire x1="79.692" y1="56.388" x2="80.48" y2="57.176" width="0.6096" layer="1"/>
 <wire x1="73.914" y1="56.388" x2="79.692" y2="56.388" width="0.6096" layer="1"/>
+<wire x1="60.85" y1="46.167" x2="60.85" y2="46.118" width="0.381" layer="1"/>
+<wire x1="60.85" y1="46.118" x2="59.6646" y2="44.9326" width="0.381" layer="1"/>
+<wire x1="59.6646" y1="44.9326" x2="59.6646" y2="41.4909" width="0.381" layer="1"/>
 </signal>
 <signal name="+5V">
@@
 <wire x1="63.881" y1="56.388" x2="63.5" y2="56.388" width="0.381" layer="16"/>
 <wire x1="64.2143" y1="51.582075" x2="64.643" y2="52.010775" width="0.381" layer="16"/>
+<contactref element="U$3" pad="P$1"/>
+<wire x1="63.39" y1="46.167" x2="63.39" y2="45.991" width="0.381" layer="1"/>
+<wire x1="62.149" y1="44.75" x2="62.149" y2="43.434" width="0.381" layer="1"/>
+<wire x1="63.39" y1="45.991" x2="62.149" y2="44.75" width="0.381" layer="1"/>
 </signal>
 <signal name="N$17">
@@
 <wire x1="65.93" y1="46.88" x2="67.437" y2="48.387" width="0.381" layer="16"/>
 <wire x1="67.183" y1="56.642" x2="67.183" y2="51.689" width="0.381" layer="16"/>
-<wire x1="63.5" y1="58.928" x2="64.516" y2="58.928" width="0.381" layer="16"/>
-<wire x1="66.802" y1="56.642" x2="67.183" y2="56.642" width="0.381" layer="16"/>
-<wire x1="64.516" y1="58.928" x2="66.802" y2="56.642" width="0.381" layer="16"/>
+<wire x1="63.5" y1="57.658" x2="65.532" y2="57.658" width="0.381" layer="16"/>
+<wire x1="66.548" y1="56.642" x2="67.183" y2="56.642" width="0.381" layer="16"/>
+<wire x1="65.532" y1="57.658" x2="66.548" y2="56.642" width="0.381" layer="16"/>
+<contactref element="U$3" pad="P$2"/>
+<wire x1="65.93" y1="46.167" x2="65.93" y2="44.848" width="0.381" layer="1"/>
+<wire x1="64.649" y1="43.567" x2="64.649" y2="43.434" width="0.381" layer="1"/>
+<wire x1="65.93" y1="44.848" x2="64.649" y2="43.567" width="0.381" layer="1"/>
 </signal>
 <signal name="N$2">
